Commit message: modified the rsp.launch file to open rviz2, joint state publisher adn joint state publisher gui

File: description/diffbot_description.urdf.xacro (robot description, xacro)
@@ -61,4 +61,7 @@
       </inertial>
     </link>
+    <gazebo reference="base_link">
+        <material>Gazebo/Orange</material>
+    </gazebo>
     <joint name="left_wheel_joint" type="continuous">
       <parent link="base_link"/>
@@ -92,4 +95,7 @@
         </inertial>
       </link>
+    <gazebo reference="left_wheel">
+        <material>Gazebo/Black</material>
+    </gazebo>
     <joint name="$right_wheel_joint" type="continuous">
       <parent link="base_link"/>
@@ -123,4 +129,7 @@
         </inertial>
      </link>
+    <gazebo reference="right_wheel">
+        <material>Gazebo/Black</material>
+    </gazebo>
     <joint name="caster_frontal_wheel_joint" type="fixed">
       <parent link="base_link"/>
@@ -152,4 +161,7 @@
         </inertial>
       </link>
+    <gazebo reference="caster_frontal_wheel">
+        <material>Gazebo/White</material>
+    </gazebo>
     <joint name="caster_rear_wheel_joint" type="fixed">
       <parent link="base_link"/>
@@ -181,3 +193,6 @@
         </inertial>
       </link>
+    <gazebo reference="caster_rear_wheel">
+        <material>Gazebo/White</material>
+    </gazebo>
 </robot>

Commit message: This has a correction to the urdf, makes the urdf the same for visual collision and inertial tags

File: description/diffbot_description.urdf.xacro (robot description, xacro)
@@ -40,5 +40,5 @@
    <link name="base_link">
     <collision>
-      <origin xyz="0 0 0" rpy="0 0 0"/>
+      <origin xyz="0 0 0.0575" rpy="0 0 0"/>
       <geometry>
         <box size="${base_width} ${base_length} ${base_height}"/>
@@ -46,5 +46,5 @@
     </collision>
     <visual>
-      <origin xyz="0 0 ${base_height/2}" rpy="0 0 0"/>
+      <origin xyz="0 0 0.0575" rpy="0 0 0"/>
       <geometry>
         <box size="${base_width} ${base_length} ${base_height}"/>
@@ -53,5 +53,5 @@
     </visual>
     <inertial>
-      <origin xyz="0 0 0" rpy="0 0 0"/>
+      <origin xyz="0 0 0.0575" rpy="0 0 0"/>
       <mass value="${base_mass}"/>
       <inertia
@@ -67,5 +67,5 @@
       <parent link="base_link"/>
       <child link="left_wheel"/>
-      <origin xyz="0 -${base_width/2} ${z_offset}" rpy="0 0 0"/>
+      <origin xyz="0 -${base_width/2} 0.015" rpy="0 0 0"/>
       <axis xyz="0 1 0"/>
       <dynamics damping="0.2"/>
@@ -101,5 +101,5 @@
       <parent link="base_link"/>
       <child link="right_wheel"/>
-      <origin xyz="0 ${base_width/2} ${z_offset}" rpy="0 0 0"/>
+      <origin xyz="0 ${base_width/2} 0.015" rpy="0 0 0"/>
       <axis xyz="0 1 0"/>
       <dynamics damping="0.2"/>
@@ -135,10 +135,10 @@
       <parent link="base_link"/>
       <child link="caster_frontal_wheel"/>
-      <origin xyz="${base_width/2 - caster_wheel_radius} 0 ${z_offset}" rpy="0 0 0"/>
+      <origin xyz="${base_width/2 - caster_wheel_radius} 0 0" rpy="0 0 0"/>
     </joint>
     <!-- caster frontal wheel Link -->
     <link name="caster_frontal_wheel">
       <collision>
-        <origin xyz="0 0 0" rpy="0 0 0"/>
+        <origin xyz="0 0 ${caster_wheel_radius}" rpy="0 0 0"/>
         <geometry>
           <sphere radius="${caster_wheel_radius}"/>
@@ -146,5 +146,5 @@
       </collision>
       <visual>
-        <origin xyz="0 0 0" rpy="0 0 0"/>
+        <origin xyz="0 0 ${caster_wheel_radius}" rpy="0 0 0"/>
         <geometry>
           <sphere radius="${caster_wheel_radius}"/>
@@ -153,5 +153,5 @@
       </visual>
       <inertial>
-        <origin xyz="0 0 0" rpy="0 0 0"/>
+        <origin xyz="0 0 ${caster_wheel_radius}" rpy="0 0 0"/>
         <mass value="${caster_wheel_mass}"/>
         <inertia
@@ -167,10 +167,10 @@
       <parent link="base_link"/>
       <child link="caster_rear_wheel"/>
-      <origin xyz="${-base_width/2 + caster_wheel_radius} 0 ${z_offset}" rpy="0 0 0"/>
+      <origin xyz="${-base_width/2 + caster_wheel_radius} 0 0" rpy="0 0 0"/>
     </joint>
     <!-- caster rear wheel Link -->
     <link name="caster_rear_wheel">
       <collision>
-        <origin xyz="0 0 0" rpy="0 0 0"/>
+        <origin xyz="0 0 ${caster_wheel_radius}" rpy="0 0 0"/>
         <geometry>
           <sphere radius="${caster_wheel_radius}"/>
@@ -178,5 +178,5 @@
       </collision>
       <visual>
-        <origin xyz="0 0 0" rpy="0 0 0"/>
+        <origin xyz="0 0 ${caster_wheel_radius}" rpy="0 0 0"/>
         <geometry>
           <sphere radius="${caster_wheel_radius}"/>
@@ -185,5 +185,5 @@
       </visual>
       <inertial>
-        <origin xyz="0 0 0" rpy="0 0 0"/>
+        <origin xyz="0 0 ${caster_wheel_radius}" rpy="0 0 0"/>
         <mass value="${caster_wheel_mass}"/>
         <inertia

Commit message: This runs the dif bot URDF, the ros2_control xacro and drives it manuall using a publisher

File: description/diffbot_description.urdf.xacro (robot description, xacro)
@@ -98,5 +98,5 @@
         <material>Gazebo/Black</material>
     </gazebo>
-    <joint name="$right_wheel_joint" type="continuous">
+    <joint name="right_wheel_joint" type="continuous">
       <parent link="base_link"/>
       <child link="right_wheel"/>

File: description/robot.urdf.xacro (robot description, xacro)
@@ -3,3 +3,4 @@
   <xacro:include filename="diffbot_description.urdf.xacro"/>
   <!--<xacro:include filename="diffbot.materials.xacro"/> -->
+  <xacro:include filename="diffbot.ros2_control.xacro"/>
 </robot>
